File: PCB/robotrev2.sch (EAGLE design)
At the start: 55 parts, among them J1 1X2-3.5MM, J2 1X2-3.5MM, P1 BSS84, P2 BSS84, U1 ATTINY861A-SU, X1 USB-MICROB, X5 USBSMD

Commit message: PCB updated to rev2.
Parts:
- removed 128: SWITCH-MOMENTARY-2-SMD-1101NE, SparkFun:SWITCH-MOMENTARY-2-SMD-1101NE
- removed J1, J2: 1X2-3.5MM, adafruit:1X2-3.5MM
- removed N1, N2: BSS123, transistor-small-signal:BSS123
- removed P1, P2: BSS84, transistor-small-signal:BSS84
- removed X1: USB-MICROB, SparkFun:USB-MICROB
- added 3: SWITCH-MOMENTARY-2-SMD-1101NE, SparkFun:SWITCH-MOMENTARY-2-SMD-1101NE
- added BATTERYENABLE: SOLDERJUMPERNO, SparkFun:SOLDERJUMPERNO
- added C1, C3: 10uF, rc-master-smd:C_0603
- added C6, C7: 100n, rc-master-smd:C_0603
- added CHARGER: (no value), led:LEDSML0603
- added IC1: 74HCT14D, 74xx-eu:74HCT14D
- added IC2: MCP73831, SparkFunNew:MCP73831
- added JP5, JP6: (no value), pinhead:PINHD-1X2
- added LEDCH: 1k, rcl:R-EU_R0603
- added R13: 1k, resistor:R-EU_R0603
- added R14: 200, resistor:R-EU_R0603
- added R15: 56, resistor:R-EU_R0603
- added RPROG: 22K, rcl:R-EU_R0603
- added USB1: USB-MICROBLARGEPAD, zak:USB-MICROBLARGEPAD
- JP1, JP2: device pinhead:PINHD-1X1 -> pinhead:PINHD-1X2
- R6: value 256 -> 256k
- U$3, U$4: value MOUNTINGHOLE1.0 -> MOUNTINGHOLE2.0; device microbuilder:MOUNTINGHOLE1.0 -> microbuilder:MOUNTINGHOLE2.0
- U$6, U$7: value MOUNTINGHOLE3.0THIN -> MOUNTINGHOLE2.0; device microbuilder:MOUNTINGHOLE3.0THIN -> microbuilder:MOUNTINGHOLE2.0
- renumbered 16 to 5, 32 to 6, 64 to 7
Connections:
- removed net 5V: 3V3.VIN, BATTERY.+, C4.1, J2.1, P1.S, P2.S, X1.VBUS, X5.VBUS
- removed net LEDX: U$1.3
- removed net OUTL: N2.D, P2.D, R6.1
- removed net OUTR: C2.+, N1.D, P1.D, R6.2
- removed net RESET: S1.2
- removed net SPEAKER: C2.-, J1.2, JP1.1
- new net LED0X: PB1.A, R2.1
- new net LED1X: PB3.A, R4.1
- new net LINE: JP6.2, R13.2, R6.2
- new net N$12: IC1C.O, R14.1
- new net N$13: C2.+, IC1D.O, IC1E.O, IC1F.O, R15.2
- new net N$14: C2.-, JP2.1, JP5.1
- new net N$15: IC1A.O, R6.1
- new net N$16: IC1B.O, R13.1
- new net N$17: R14.2, R15.1
- new net N$18: CHARGER.C, IC2.STAT
- new net N$31: IC2.PROG, RPROG.2
- new net N$35: CHARGER.A, LEDCH.1
- new net VBAT: 3V3.VIN, BATTERY.+, BATTERYENABLE.1, C3.1, C4.1, IC1P.VCC, IC2.VBAT, JP1.1
- new net VBUS: BATTERYENABLE.2, C1.1, IC2.VIN, LEDCH.2, USB1.VBUS, X5.VBUS
- net 128: now also 8.1; no longer 128.1
- net 4: now also 3.1; no longer 4.1
- net 8: now also 4.1; no longer 8.1
- net GND: now also 3.2, C1.2, C3.2, C6.1, C7.1, IC1P.GND, IC2.VSS, JP1.2, JP2.2, JP5.2, JP6.1, RPROG.1, USB1.GND; no longer 128.2, J1.1, J2.2, JP2.1, N1.S, N2.S, X1.GND
- net LED: now also U$1.3; no longer PB1.A, PB3.A, R2.1, R4.1
- net PB1: now also IC1A.I, IC1C.I, R4.2; no longer N1.G, P1.G
- net PB3: now also IC1B.I, IC1D.I, IC1E.I, IC1F.I; no longer N2.G, P2.G, R4.2
- net RES: now also S1.2
- net VCC: now also C6.2, C7.2
Other:
- moved on the sheet: 4, 8, C2, C4, R6, U$1, U$9
